File: Electronics/KiCad Mini Projects/6 Integrated Air Quality & Environmental Monitor/6 Integrated Air Quality & Environmental Monitor.kicad_pcb (KiCad board)
At the start: 2 copper layers, 157 x 53.3 mm, 21 parts, among them J1 Power, J10 MQ4, J11 MQ5, J12 MQ6, J13 MQ7, J14 MQ8, J15 MQ9, J16 MQ135, J17 MQ139, J18 KY028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

Commit message: KiCad Mini Projects files
Parts:
- J10: value MQ4 -> MQ2; footprint Connector_PinSocket_2.54mm:PinSocket_1x04_P2.54mm_Vertical -> My Library:MQ_Module_Vertical
- J11: value MQ5 -> MQ3; footprint Connector_PinSocket_2.54mm:PinSocket_1x04_P2.54mm_Vertical -> My Library:MQ_Module_Vertical
- J12: value MQ6 -> MQ135; footprint Connector_PinSocket_2.54mm:PinSocket_1x04_P2.54mm_Vertical -> My Library:MQ_Module_Vertical
- J13: value MQ7 -> MQ4
- J14: value MQ8 -> MQ5
- J15: value MQ9 -> MQ6; footprint Connector_PinSocket_2.54mm:PinSocket_1x04_P2.54mm_Vertical -> My Library:MQ_Module_Vertical
- J16: value MQ135 -> MQ7; footprint Connector_PinSocket_2.54mm:PinSocket_1x04_P2.54mm_Vertical -> My Library:MQ_Module_Vertical
- J17: value MQ139 -> MQ8; footprint Connector_PinSocket_2.54mm:PinSocket_1x04_P2.54mm_Vertical -> My Library:MQ_Module_Vertical
- J18: value KY028 -> MQ9
- J19: value DHT11 -> MQ139; footprint Connector_PinSocket_2.54mm:PinSocket_1x03_P2.54mm_Vertical -> Connector_PinHeader_2.54mm:PinHeader_1x04_P2.54mm_Vertical
- J20: value DHT11 -> KY028; footprint Connector_PinSocket_2.54mm:PinSocket_1x03_P2.54mm_Vertical -> Connector_PinSocket_2.54mm:PinSocket_1x04_P2.54mm_Vertical
- J8: value MQ2 -> DHT11; footprint Connector_PinSocket_2.54mm:PinSocket_1x04_P2.54mm_Vertical -> Connector_PinSocket_2.54mm:PinSocket_1x03_P2.54mm_Vertical
- J9: value MQ3 -> DHT11; footprint Connector_PinSocket_2.54mm:PinSocket_1x04_P2.54mm_Vertical -> Connector_PinSocket_2.54mm:PinSocket_1x03_P2.54mm_Vertical
- moved J20 167.0 mm to (272.8, 87.2), turned to 0 degrees
- moved J8 78.7 mm to (204.9, 50.1)
- moved J13 73.9 mm to (254.7, 96.5), turned to 90 degrees
- moved J18 53.2 mm to (270.5, 76.6), turned to 180 degrees
- moved J15 51.3 mm to (160.2, 84.7)
- moved J19 47.8 mm to (207.6, 97.9)
- moved J16 41.2 mm to (197.2, 84.3)
- moved J14 39.1 mm to (220.9, 97.5)
- moved J12 32.0 mm to (131.9, 84.4), turned to 0 degrees
- moved J9 26.2 mm to (108.8, 50.8), turned to -90 degrees
- moved J10 21.6 mm to (149.0, 62.5)
- moved J7 19.4 mm to (259.9, 53.1), turned to 180 degrees
- moved J11 13.4 mm to (185.3, 62.8)
- moved J17 8.08 mm to (230.0, 75.1)
- moved J21 1.19 mm to (230.0, 50.0), turned to -90 degrees
Connections:
- J10 pad 4: /A3 -> /A0
- J11 pad 4: /A4 -> /A1
- J12 pad 4: /A5 -> /A2
- J13 pad 4: /A6 -> /A3
- J14 pad 4: /A7 -> /A4
- J15 pad 4: /A8 -> /A5
- J16 pad 4: /A2 -> /A6
- J17 pad 4: /A9 -> /A7
- J18 pad 1: /A11 -> +5V
- J18 pad 3: +5V -> unconnected-(J18-Pin_3-Pad3)
- J18 pad 4: unconnected-(J18-Pin_4-Pad4) -> /A8
- J19 pad 2: /D4 -> GND
- J19 pad 3: GND -> unconnected-(J19-Pin_3-Pad3)
- J20 pad 1: +5V -> /A11
- J20 pad 2: /D2 -> GND
- J20 pad 3: GND -> +5V
- J8 pad 2: GND -> /D4
- J8 pad 3: unconnected-(J8-Pin_3-Pad3) -> GND
- J9 pad 2: GND -> /D2
- J9 pad 3: unconnected-(J9-Pin_3-Pad3) -> GND
Routing:
- net /A1: track 36.7 -> 137.2 mm
- net +5V: track 425.8 -> 517.2 mm
- net /A0: track 10.2 -> 89.3 mm
- net /A3: track 37.3 -> 106.0 mm
- net /A8: track 42.8 -> 108.8 mm
- net /A11: track 42.3 -> 95.8 mm
- net /A7: track 23.8 -> 72.9 mm
- net /A9: track 67.4 -> 24.7 mm
- net /A4: track 55.9 -> 68.9 mm
- net /A2: track 13.0 -> 24.5 mm
- net /A6: track 28.8 -> 38.2 mm
- net /SCL/21: track 49.0 -> 42.9 mm
- net /SDA/20: track 51.6 -> 48.3 mm
- net /A5: track 10.5 -> 8.74 mm
- net /D2: track 47.2 -> 45.7 mm
Other:
- board size 157 x 53.3 mm -> 178 x 53.3 mm
- board text added: "A"
- board text added: "A9"
- board text added: "D"
- board text added: "D2"
- board text added: "D4"
- board text added: "Digital"
- board text added: "GND"
- board text added: "ICSP"
- board text added: "SCL"
- board text added: "SDA"
- board text added: "x"
